Commit message: Add launch file and update start script
This commit adds a new launch file `robot_description.launch.py` for
loading the robot's URDF description. It also updates the `start.sh`
script to include the execution of this launch file before starting
other ROS nodes. This ensures that the robot's state is published
correctly before any other components are initialized.

File: data/src/edutracker_description/urdf/robot.urdf.xacro (robot description, xacro)
@@ -1,18 +1,16 @@
-<?xml version="1.0"?>
+<?xml version="1.0" ?>
 <robot xmlns:xacro="http://ros.org/wiki/xacro" name="edutracker">
   <!-- ====== ПАРАМЕТРЫ ====== -->
-  <xacro:property name="body_radius" value="0.125"/>
-  <xacro:property name="body_height" value="0.05"/>
-  <xacro:property name="wheel_radius" value="0.0325"/>
-  <xacro:property name="wheel_width" value="0.02"/>
+  <xacro:property name="body_radius" value="0.125" />
+  <xacro:property name="body_height" value="0.05" />
+  <xacro:property name="wheel_radius" value="0.0325" />
+  <xacro:property name="wheel_width" value="0.02" />
   <!-- ====== BASE ====== -->
   <link name="base_link">
     <visual>
       <geometry>
-        <cylinder
-          radius="${body_radius}"
-          length="${body_height}"/>
+        <cylinder radius="${body_radius}" length="${body_height}" />
       </geometry>
-      <origin xyz="0 0 0"/>
+      <origin xyz="0 0 0" />
     </visual>
   </link>
@@ -21,14 +19,14 @@
     <visual>
       <geometry>
-        <cylinder radius="0.035" length="0.05"/>
+        <cylinder radius="0.035" length="0.05" />
       </geometry>
-      <origin xyz="0 0 0"/>
+      <origin xyz="0 0 0" />
     </visual>
   </link>
   <joint name="laser_joint" type="fixed">
-    <parent link="base_link"/>
-    <child link="laser_link"/>
+    <parent link="base_link" />
+    <child link="laser_link" />
     <!-- 25 см выше базы -->
-    <origin xyz="0 0 0.25"/>
+    <origin xyz="0 0 0.25" />
   </joint>
   <!-- ====== CAMERA ====== -->
@@ -36,13 +34,13 @@
     <visual>
       <geometry>
-        <box size="0.04 0.04 0.03"/>
+        <box size="0.04 0.04 0.03" />
       </geometry>
     </visual>
   </link>
   <joint name="camera_joint" type="fixed">
-    <parent link="base_link"/>
-    <child link="camera_link"/>
+    <parent link="base_link" />
+    <child link="camera_link" />
     <!-- камера чуть сбоку и выше -->
-    <origin xyz="0.05 0 0.20"/>
+    <origin xyz="0.05 0 0.20" />
   </joint>
   <!-- ====== КОЛЁСА ====== -->
@@ -50,32 +48,28 @@
     <visual>
       <geometry>
-        <cylinder
-          radius="${wheel_radius}"
-          length="${wheel_width}"/>
+        <cylinder radius="${wheel_radius}" length="${wheel_width}" />
       </geometry>
-      <origin rpy="1.5708 0 0"/>
+      <origin rpy="1.5708 0 0" />
     </visual>
   </link>
   <joint name="left_wheel_joint" type="continuous">
-    <parent link="base_link"/>
-    <child link="left_wheel_link"/>
-    <origin xyz="0 0.13 0"/>
-    <axis xyz="0 1 0"/>
+    <parent link="base_link" />
+    <child link="left_wheel_link" />
+    <origin xyz="0 0.13 0" />
+    <axis xyz="0 1 0" />
   </joint>
   <link name="right_wheel_link">
     <visual>
       <geometry>
-        <cylinder
-          radius="${wheel_radius}"
-          length="${wheel_width}"/>
+        <cylinder radius="${wheel_radius}" length="${wheel_width}" />
       </geometry>
-      <origin rpy="1.5708 0 0"/>
+      <origin rpy="1.5708 0 0" />
     </visual>
   </link>
   <joint name="right_wheel_joint" type="continuous">
-    <parent link="base_link"/>
-    <child link="right_wheel_link"/>
-    <origin xyz="0 -0.13 0"/>
-    <axis xyz="0 1 0"/>
+    <parent link="base_link" />
+    <child link="right_wheel_link" />
+    <origin xyz="0 -0.13 0" />
+    <axis xyz="0 1 0" />
   </joint>
 </robot>

Commit message: fix model

File: data/src/edutracker_description/urdf/robot.urdf.xacro (robot description, xacro)
@@ -2,17 +2,23 @@
 <robot xmlns:xacro="http://ros.org/wiki/xacro" name="edutracker">
   <!-- ====== ПАРАМЕТРЫ ====== -->
-  <xacro:property name="body_radius" value="0.125" />
-  <xacro:property name="body_height" value="0.05" />
+  <xacro:property name="body_radius" value="0.0775" />
+  <xacro:property name="body_height" value="0.245" />
   <xacro:property name="wheel_radius" value="0.0325" />
-  <xacro:property name="wheel_width" value="0.02" />
+  <xacro:property name="wheel_width" value="0.027" />
   <!-- ====== BASE ====== -->
-  <link name="base_link">
-    <visual>
-      <geometry>
-        <cylinder radius="${body_radius}" length="${body_height}" />
-      </geometry>
-      <origin xyz="0 0 0" />
-    </visual>
+  <link name="base_link"/>
+  <link name="body_link">
+      <visual>
+        <geometry>
+          <cylinder radius="${body_radius}" length="${body_height}" />
+        </geometry>
+        <origin xyz="-0.047 0 0.1225" />
+      </visual>
   </link>
+  <joint name="body_joint" type="fixed">
+    <parent link="base_link"/>
+    <child link="body_link"/>
+    <origin xyz="0 0 0"/>
+  </joint>
   <!-- ====== LIDAR ====== -->
   <link name="laser_link">
@@ -28,5 +34,5 @@
     <child link="laser_link" />
     <!-- 25 см выше базы -->
-    <origin xyz="0 0 0.25" />
+    <origin xyz="-0.047 0 0.2755" />
   </joint>
   <!-- ====== CAMERA ====== -->
@@ -56,5 +62,5 @@
     <parent link="base_link" />
     <child link="left_wheel_link" />
-    <origin xyz="0 0.13 0" />
+    <origin xyz="0 0.1155 0" />
     <axis xyz="0 1 0" />
   </joint>
@@ -70,5 +76,5 @@
     <parent link="base_link" />
     <child link="right_wheel_link" />
-    <origin xyz="0 -0.13 0" />
+    <origin xyz="0 -0.1155 0" />
     <axis xyz="0 1 0" />
   </joint>

Commit message: add material

File: data/src/edutracker_description/urdf/robot.urdf.xacro (robot description, xacro)
@@ -14,4 +14,5 @@
         </geometry>
         <origin xyz="-0.047 0 0.1225" />
+        <material name="gray"/>
       </visual>
   </link>
@@ -28,4 +29,5 @@
       </geometry>
       <origin xyz="0 0 0" />
+      <material name="gray"/>
     </visual>
   </link>
@@ -42,4 +44,5 @@
         <box size="0.04 0.04 0.03" />
       </geometry>
+      <material name="gray"/>
     </visual>
   </link>
@@ -57,4 +60,5 @@
       </geometry>
       <origin rpy="1.5708 0 0" />
+      <material name="gray"/>
     </visual>
   </link>
@@ -71,4 +75,5 @@
       </geometry>
       <origin rpy="1.5708 0 0" />
+      <material name="gray"/>
     </visual>
   </link>

Commit message: add materials

File: data/src/edutracker_description/urdf/robot.urdf.xacro (robot description, xacro)
@@ -6,4 +6,10 @@
   <xacro:property name="wheel_radius" value="0.0325" />
   <xacro:property name="wheel_width" value="0.027" />
+  <material name="green">
+    <color rgba="0 0.6 0 1"/>
+  </material>
+  <material name="black">
+    <color rgba="0 0 0 1"/>
+  </material>
   <!-- ====== BASE ====== -->
   <link name="base_link"/>
@@ -14,5 +20,5 @@
         </geometry>
         <origin xyz="-0.047 0 0.1225" />
-        <material name="gray"/>
+        <material name="green"/>
       </visual>
   </link>
@@ -29,5 +35,5 @@
       </geometry>
       <origin xyz="0 0 0" />
-      <material name="gray"/>
+      <material name="black"/>
     </visual>
   </link>
@@ -44,5 +50,5 @@
         <box size="0.04 0.04 0.03" />
       </geometry>
-      <material name="gray"/>
+      <material name="black"/>
     </visual>
   </link>
@@ -60,5 +66,5 @@
       </geometry>
       <origin rpy="1.5708 0 0" />
-      <material name="gray"/>
+      <material name="black"/>
     </visual>
   </link>
@@ -75,5 +81,5 @@
       </geometry>
       <origin rpy="1.5708 0 0" />
-      <material name="gray"/>
+      <material name="black"/>
     </visual>
   </link>

Commit message: Update robot.urdf.xacro

File: data/src/edutracker_description/urdf/robot.urdf.xacro (robot description, xacro)
@@ -7,5 +7,5 @@
   <xacro:property name="wheel_width" value="0.027" />
   <material name="green">
-    <color rgba="0 0.6 0 1"/>
+    <color rgba="0 0.6 0 0.8"/>
   </material>
   <material name="black">
@@ -48,5 +48,5 @@
     <visual>
       <geometry>
-        <box size="0.04 0.04 0.03" />
+        <box size="0.01 0.38 0.30" />
       </geometry>
       <material name="black"/>
@@ -57,5 +57,5 @@
     <child link="camera_link" />
     <!-- камера чуть сбоку и выше -->
-    <origin xyz="0.05 0 0.20" />
+    <origin xyz="-0.01 0 0.203" />
   </joint>
   <!-- ====== КОЛЁСА ====== -->

Commit message: fix new form factor!

File: data/src/edutracker_description/urdf/robot.urdf.xacro (robot description, xacro)
@@ -7,24 +7,28 @@
   <xacro:property name="wheel_width" value="0.027" />
   <material name="green">
-    <color rgba="0 0.6 0 0.8"/>
+    <color rgba="0 0.6 0 0.8" />
   </material>
   <material name="black">
-    <color rgba="0 0 0 1"/>
+    <color rgba="0 0 0 1" />
   </material>
   <!-- ====== BASE ====== -->
-  <link name="base_link"/>
+  <link name="base_link" />
   <link name="body_link">
       <visual>
         <geometry>
-          <cylinder radius="${body_radius}" length="${body_height}" />
+          <!-- <cylinder radius="${body_radius}" length="${body_height}" /> -->
+          <mesh
+                      filename="package://edutracker_description/meshes/base.stl"
+                      scale="0.001 0.001 0.001"
+                  />
         </geometry>
         <origin xyz="-0.047 0 0.1225" />
-        <material name="green"/>
+        <material name="green" />
       </visual>
   </link>
   <joint name="body_joint" type="fixed">
-    <parent link="base_link"/>
-    <child link="body_link"/>
-    <origin xyz="0 0 0"/>
+    <parent link="base_link" />
+    <child link="body_link" />
+    <origin xyz="0 0 0" />
   </joint>
   <!-- ====== LIDAR ====== -->
@@ -32,8 +36,12 @@
     <visual>
       <geometry>
-        <cylinder radius="0.035" length="0.05" />
+        <!-- <cylinder radius="0.035" length="0.05" /> -->
+        <mesh
+                    filename="package://edutracker_description/meshes/lidar.stl"
+                    scale="0.001 0.001 0.001"
+                />
       </geometry>
       <origin xyz="0 0 0" />
-      <material name="black"/>
+      <material name="black" />
     </visual>
   </link>
@@ -48,7 +56,7 @@
     <visual>
       <geometry>
-        <box size="0.01 0.38 0.30" />
+        <box size="0.01 0.038 0.03" />
       </geometry>
-      <material name="black"/>
+      <material name="black" />
     </visual>
   </link>
@@ -63,8 +71,12 @@
     <visual>
       <geometry>
-        <cylinder radius="${wheel_radius}" length="${wheel_width}" />
+        <!-- <cylinder radius="${wheel_radius}" length="${wheel_width}" /> -->
+        <mesh
+                    filename="package://edutracker_description/meshes/wheel.stl"
+                    scale="0.001 0.001 0.001"
+                />
       </geometry>
       <origin rpy="1.5708 0 0" />
-      <material name="black"/>
+      <material name="black" />
     </visual>
   </link>
@@ -78,8 +90,12 @@
     <visual>
       <geometry>
-        <cylinder radius="${wheel_radius}" length="${wheel_width}" />
+        <!-- <cylinder radius="${wheel_radius}" length="${wheel_width}" /> -->
+        <mesh
+                    filename="package://edutracker_description/meshes/wheel.stl"
+                    scale="0.001 0.001 0.001"
+                />
       </geometry>
-      <origin rpy="1.5708 0 0" />
-      <material name="black"/>
+      <origin rpy="-1.5708 0 0" />
+      <material name="black" />
     </visual>
   </link>

Commit message: Update robot.urdf.xacro

File: data/src/edutracker_description/urdf/robot.urdf.xacro (robot description, xacro)
@@ -17,9 +17,9 @@
       <visual>
         <geometry>
-          <!-- <cylinder radius="${body_radius}" length="${body_height}" /> -->
-          <mesh
+          <cylinder radius="${body_radius}" length="${body_height}" />
+          <!-- <mesh
                       filename="package://edutracker_description/meshes/base.stl"
                       scale="0.001 0.001 0.001"
-                  />
+                  /> -->
         </geometry>
         <origin xyz="-0.047 0 0.1225" />
@@ -36,9 +36,9 @@
     <visual>
       <geometry>
-        <!-- <cylinder radius="0.035" length="0.05" /> -->
-        <mesh
+        <cylinder radius="0.035" length="0.05" />
+        <!-- <mesh
                     filename="package://edutracker_description/meshes/lidar.stl"
                     scale="0.001 0.001 0.001"
-                />
+                /> -->
       </geometry>
       <origin xyz="0 0 0" />
@@ -71,9 +71,9 @@
     <visual>
       <geometry>
-        <!-- <cylinder radius="${wheel_radius}" length="${wheel_width}" /> -->
-        <mesh
+        <cylinder radius="${wheel_radius}" length="${wheel_width}" />
+        <!-- <mesh
                     filename="package://edutracker_description/meshes/wheel.stl"
                     scale="0.001 0.001 0.001"
-                />
+                /> -->
       </geometry>
       <origin rpy="1.5708 0 0" />
@@ -90,9 +90,9 @@
     <visual>
       <geometry>
-        <!-- <cylinder radius="${wheel_radius}" length="${wheel_width}" /> -->
-        <mesh
+        <cylinder radius="${wheel_radius}" length="${wheel_width}" />
+        <!-- <mesh
                     filename="package://edutracker_description/meshes/wheel.stl"
                     scale="0.001 0.001 0.001"
-                />
+                /> -->
       </geometry>
       <origin rpy="-1.5708 0 0" />

Commit message: 1

File: data/src/edutracker_description/urdf/robot.urdf.xacro (robot description, xacro)
@@ -3,5 +3,5 @@
   <!-- ====== ПАРАМЕТРЫ ====== -->
   <xacro:property name="body_radius" value="0.0775" />
-  <xacro:property name="body_height" value="0.245" />
+  <xacro:property name="body_height" value="0.230" />
   <xacro:property name="wheel_radius" value="0.0325" />
   <xacro:property name="wheel_width" value="0.027" />
@@ -50,5 +50,5 @@
     <child link="laser_link" />
     <!-- 25 см выше базы -->
-    <origin xyz="-0.047 0 0.2755" />
+    <origin xyz="-0.047 0 0.260" />
   </joint>
   <!-- ====== CAMERA ====== -->
